File: circuit_ESP32C3_Xiao/ESP32C3_Xiao_wireless_DAP.kicad_pcb (KiCad board)
At the start: 2 copper layers, 70 x 35 mm, 42 parts, among them J1 Cortex Debug 10pin connector, J2 ARM Standard JTAG, J3 Cortex Debug 10pin connector, J4 Conn_01x02, J6 Serial, Q1 YJL2304A, U1 XIAO-ESP32-C3-SMD, U2 AP1117-ADJ

Commit message: Update ESP32-C3 VTarget hardware design
Record the current ESP32-C3 XIAO schematic and PCB updates for the VTarget circuit.
Parts:
- C2: value 10nF -> 10uF /16V
- R4: value 39k -> 22k
- R5: value 10k -> 43k
Connections:
- net Net-(U2-ADJ) renamed /Vadj
Changed lines of the file:
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@@
 	(net 30 "unconnected-(U1-MTCK-Pad22)")
 	(net 31 "/TDI")
-	(net 32 "Net-(U2-ADJ)")
+	(net 32 "/Vadj")
 	(net 33 "Net-(D1-K)")
 	(net 34 "Net-(D2-K)")
@@
 			(layers "F.Cu" "F.Mask" "F.Paste")
 			(roundrect_rratio 0.25)
-			(net 32 "Net-(U2-ADJ)")
+			(net 32 "/Vadj")
 			(pintype "passive")
 		)
@@
 			)
 		)
-		(property "Value" "10nF"
+		(property "Value" "10uF /16V"
 			(at 0 1.43 270)
 			(unlocked yes)
@@
 			)
 		)
-		(property "Value" "39k"
+		(property "Value" "22k"
 			(at 0 1.43 0)
 			(unlocked yes)
@@
 			)
 		)
-		(property "Value" "10k"
+		(property "Value" "43k"
 			(at 0 1.43 90)
 			(unlocked yes)
@@
 			(layers "F.Cu" "F.Mask" "F.Paste")
 			(roundrect_rratio 0.25)
-			(net 32 "Net-(U2-ADJ)")
+			(net 32 "/Vadj")
 			(pintype "passive")
 		)
@@
 			(layers "F.Cu" "F.Mask" "F.Paste")
 			(roundrect_rratio 0.25)
-			(net 32 "Net-(U2-ADJ)")
+			(net 32 "/Vadj")
 			(pintype "passive")
 		)
@@
 			(layers "F.Cu" "F.Mask" "F.Paste")
 			(roundrect_rratio 0.25)
-			(net 32 "Net-(U2-ADJ)")
+			(net 32 "/Vadj")
 			(pinfunction "ADJ")
 			(pintype "input")
@@
 			(layers "F.Cu" "F.Mask" "F.Paste")
 			(roundrect_rratio 0.25)
-			(net 32 "Net-(U2-ADJ)")
+			(net 32 "/Vadj")
 			(pintype "passive")
 		)
@@
 	(gr_line
 		(start 111.2784 70.3032)
-		(end 145.2784 70.3032)
+		(end 111.2784 84.3032)
 		(stroke
 			(width 0.15)
@@
 	)
 	(gr_line
-		(start 134.3672 84.3032)
-		(end 134.3672 58.6032)
+		(start 111.2784 70.3032)
+		(end 145.2784 70.3032)
 		(stroke
 			(width 0.15)
-			(type default)
+			(type solid)
 		)
 		(layer "Cmts.User")
@@
 	)
 	(gr_line
-		(start 145.2784 70.3032)
-		(end 145.2784 98.3532)
+		(start 111.2784 98.3032)
+		(end 145.2672 98.3032)
 		(stroke
 			(width 0.15)
@@
 	)
 	(gr_line
-		(start 111.2784 98.3032)
-		(end 145.2672 98.3032)
+		(start 134.3672 84.3032)
+		(end 84.5672 84.3032)
 		(stroke
 			(width 0.15)
@@
 	)
 	(gr_line
-		(start 169.3672 101.8032)
-		(end 99.3672 66.8032)
+		(start 134.3672 84.3032)
+		(end 134.3672 58.6032)
 		(stroke
 			(width 0.15)
@@
 	)
 	(gr_line
-		(start 169.3672 66.8032)
-		(end 99.3672 101.8032)
+		(start 134.3672 84.3032)
+		(end 134.3672 116.6032)
 		(stroke
 			(width 0.15)
@@
 	(gr_line
 		(start 134.3672 84.3032)
-		(end 134.3672 116.6032)
+		(end 187.7672 84.3032)
 		(stroke
 			(width 0.15)
@@
 	)
 	(gr_line
-		(start 111.2784 70.3032)
-		(end 111.2784 84.3032)
+		(start 145.2784 70.3032)
+		(end 145.2784 98.3532)
 		(stroke
 			(width 0.15)
-			(type solid)
+			(type default)
 		)
 		(layer "Cmts.User")
 	)
 	(gr_line
-		(start 134.3672 84.3032)
-		(end 84.5672 84.3032)
+		(start 169.3672 66.8032)
+		(end 99.3672 101.8032)
 		(stroke
 			(width 0.15)
@@
 	)
 	(gr_line
-		(start 134.3672 84.3032)
-		(end 187.7672 84.3032)
+		(start 169.3672 101.8032)
+		(end 99.3672 66.8032)
 		(stroke
 			(width 0.15)
@@
 		(layer "Edge.Cuts")
 	)
-	(gr_text "VTarget"
-		(at 137.9172 79.3532 0)
+	(gr_text "Vref"
+		(at 145.2172 89.8532 0)
 		(layer "F.SilkS")
 		(effects
 			(font
-				(size 1.2 1.2)
-				(thickness 0.2)
+				(size 0.8 0.8)
+				(thickness 0.15)
+				(bold yes)
 			)
 			(justify left bottom)
 		)
 	)
-	(gr_text "VTarget"
-		(at 145.2172 95.8532 0)
+	(gr_text "GND"
+		(at 145.2172 91.3532 0)
 		(layer "F.SilkS")
 		(effects
@@
 		)
 	)
-	(gr_text "RX"
-		(at 145.2172 94.3532 0)
+	(gr_text "TX"
+		(at 145.2172 92.8532 0)
 		(layer "F.SilkS")
 		(effects
@@
 		)
 	)
-	(gr_text "TDO"
-		(at 160.6672 95.8032 0)
+	(gr_text "RX"
+		(at 145.2172 94.3532 0)
 		(layer "F.SilkS")
 		(effects
@@
 		)
 	)
-	(gr_text "nRST"
-		(at 160.6672 98.8032 0)
+	(gr_text "VTarget"
+		(at 145.2172 95.8532 0)
 		(layer "F.SilkS")
 		(effects
@@
 		)
 	)
-	(gr_text "VTref"
-		(at 132.8672 74.7032 0)
+	(gr_text "TMS"
+		(at 160.6672 92.8032 0)
 		(layer "F.SilkS")
 		(effects
 			(font
-				(size 1.2 1.2)
-				(thickness 0.2)
+				(size 0.8 0.8)
+				(thickness 0.15)
+				(bold yes)
 			)
 			(justify left bottom)
 		)
 	)
-	(gr_text "TX"
-		(at 132.1172 91.6532 0)
+	(gr_text "TCK"
+		(at 160.6672 94.3032 0)
 		(layer "F.SilkS")
 		(effects
 			(font
-				(size 2 1.4)
-				(thickness 0.3)
+				(size 0.8 0.8)
+				(thickness 0.15)
 				(bold yes)
 			)
@@
 		)
 	)
-	(gr_text "TX"
-		(at 145.2172 92.8532 0)
+	(gr_text "TDO"
+		(at 160.6672 95.8032 0)
 		(layer "F.SilkS")
 		(effects
@@
 		)
 	)
-	(gr_text "uC_VTref"
-		(at 123.6672 100.3032 0)
+	(gr_text "TDI"
+		(at 160.6672 97.3032 0)
 		(layer "F.SilkS")
 		(effects
 			(font
-				(size 2 1.4)
-				(thickness 0.3)
+				(size 0.8 0.8)
+				(thickness 0.15)
 				(bold yes)
 			)
@@
 		)
 	)
-	(gr_text "TMS"
-		(at 160.6672 92.8032 0)
+	(gr_text "nRST"
+		(at 160.6672 98.8032 0)
 		(layer "F.SilkS")
 		(effects
@@
 		)
 	)
-	(gr_text "TCK"
-		(at 160.6672 94.3032 0)
+	(gr_text "VTref"
+		(at 132.8672 74.7032 0)
 		(layer "F.SilkS")
 		(effects
 			(font
-				(size 0.8 0.8)
-				(thickness 0.15)
-				(bold yes)
+				(size 1.2 1.2)
+				(thickness 0.2)
 			)
 			(justify left bottom)
 		)
 	)
-	(gr_text "Vref"
-		(at 145.2172 89.8532 0)
+	(gr_text "VTarget"
+		(at 137.9172 79.3532 0)
 		(layer "F.SilkS")
 		(effects
 			(font
-				(size 0.8 0.8)
-				(thickness 0.15)
-				(bold yes)
+				(size 1.2 1.2)
+				(thickness 0.2)
 			)
 			(justify left bottom)
 		)
 	)
-	(gr_text "TDI"
-		(at 160.6672 97.3032 0)
+	(gr_text "uC_VTref"
+		(at 123.6672 100.3032 0)
 		(layer "F.SilkS")
 		(effects
 			(font
-				(size 0.8 0.8)
-				(thickness 0.15)
+				(size 2 1.4)
+				(thickness 0.3)
 				(bold yes)
 			)
@@
 		)
 	)
-	(gr_text "GND"
-		(at 145.2172 91.3532 0)
+	(gr_text "TX"
+		(at 132.1172 91.6532 0)
 		(layer "F.SilkS")
 		(effects
 			(font
-				(size 0.8 0.8)
-				(thickness 0.15)
+				(size 2 1.4)
+				(thickness 0.3)
 				(bold yes)
 			)
@@
 		)
 	)
-	(gr_text "Pin 7: UART_RX  Pin 8: TDI"
-		(at 135.2172 78.7532 0)
+	(gr_text "13:TDO 14:GND 15:nRST 16:GND 17:RX 18:GND"
+		(at 112.800533 85.5032 0)
 		(layer "B.SilkS")
 		(effects
@@
 		)
 	)
-	(gr_text "Pin 3: GND      Pin 4: TCK/SWCLK"
-		(at 133.050533 76.1532 0)
+	(gr_text "1:VTref 2:VTref 3:nTRST 4:GND 5:TDI 6:GND"
+		(at 113.917201 82.9032 0)
 		(layer "B.SilkS")
 		(effects
@@
 		)
 	)
-	(gr_text "Pin 5: UART_TX  Pin 6: TDO/SWO"
-		(at 133.633867 77.4532 0)
+	(gr_text "19:VTarget 20:VTref (TX:11 RX:17)"
+		(at 116.183866 86.8032 0)
 		(layer "B.SilkS")
 		(effects
@@
 		)
 	)
-	(gr_text "10-PIN CORTEX DEBUG (J1/J3)"
-		(at 127.801959 72.8532 0)
+	(gr_text "Pin 3: GND      Pin 4: TCK/SWCLK"
+		(at 133.050533 76.1532 0)
 		(layer "B.SilkS")
 		(effects
 			(font
-				(size 1.2 1.2)
-				(thickness 0.2)
-				(bold yes)
+				(size 0.7 0.7)
+				(thickness 0.12)
 			)
 			(justify mirror)
 		)
 	)
-	(gr_text "20-PIN ARM JTAG (J2)"
-		(at 114.768627 80.9032 0)
+	(gr_text "Pin 1: VTref    Pin 2: TMS/SWDIO"
+		(at 133.433867 74.8532 0)
 		(layer "B.SilkS")
 		(effects
 			(font
-				(size 1.2 1.2)
-				(thickness 0.2)
-				(bold yes)
+				(size 0.7 0.7)
+				(thickness 0.12)
 			)
 			(justify mirror)
 		)
 	)
-	(gr_text "19:VTarget 20:VTref (TX:11 RX:17)"
-		(at 116.183866 86.8032 0)
+	(gr_text "Pin 5: UART_TX  Pin 6: TDO/SWO"
+		(at 133.633867 77.4532 0)
 		(layer "B.SilkS")
 		(effects
@@
 		)
 	)
-	(gr_text "13:TDO 14:GND 15:nRST 16:GND 17:RX 18:GND"
-		(at 112.800533 85.5032 0)
+	(gr_text "Pin 9: VTarget  Pin 10: nRST"
+		(at 134.7172 80.0532 0)
 		(layer "B.SilkS")
 		(effects
@@
 		)
 	)
-	(gr_text "Pin 1: VTref    Pin 2: TMS/SWDIO"
-		(at 133.433867 74.8532 0)
+	(gr_text "Pin 7: UART_RX  Pin 8: TDI"
+		(at 135.2172 78.7532 0)
 		(layer "B.SilkS")
 		(effects
@@
 		)
 	)
-	(gr_text "Pin 9: VTarget  Pin 10: nRST"
-		(at 134.7172 80.0532 0)
+	(gr_text "20-PIN ARM JTAG (J2)"
+		(at 114.768627 80.9032 0)
 		(layer "B.SilkS")
 		(effects
 			(font
-				(size 0.7 0.7)
-				(thickness 0.12)
+				(size 1.2 1.2)
+				(thickness 0.2)
+				(bold yes)
 			)
 			(justify mirror)
 		)
 	)
-	(gr_text "1:VTref 2:VTref 3:nTRST 4:GND 5:TDI 6:GND"
-		(at 113.917201 82.9032 0)
+	(gr_text "10-PIN CORTEX DEBUG (J1/J3)"
+		(at 127.801959 72.8532 0)
 		(layer "B.SilkS")
 		(effects
 			(font
-				(size 0.7 0.7)
-				(thickness 0.12)
+				(size 1.2 1.2)
+				(thickness 0.2)
+				(bold yes)
 			)
 			(justify mirror)

Commit message: Calibrate VTarget PWM control range
Map VTarget commands to the DMM-verified operating window, update the ESP32-C3 board values, refresh test curves, and document the calibration results.
Parts:
- C2: value 10uF /16V -> 10uF /25V
- R4: value 22k -> 100R
Changed lines of the file:
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@@
 			)
 		)
-		(property "Value" "10uF /16V"
+		(property "Value" "10uF /25V"
 			(at 0 1.43 270)
 			(unlocked yes)
@@
 			)
 		)
-		(property "Value" "22k"
+		(property "Value" "100R"
 			(at 0 1.43 0)
 			(unlocked yes)

Commit message: Update KiCad schematic, PCB, and iBOM
Sync ESP32-C3 XIAO KiCad schematic, PCB, and interactive BOM with the R4/R5/C2 calibration hardware.
Parts:
- R1: value 12k -> 1.2k
- R3: value 27k -> 2.7k
- R4: value 100R -> 22k
Changed lines of the file:
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@@
 			)
 		)
-		(property "Value" "100R"
+		(property "Value" "22k"
 			(at 0 1.43 0)
 			(unlocked yes)
@@
 			)
 		)
-		(property "Value" "12k"
+		(property "Value" "1.2k"
 			(at 0 1.43 90)
 			(unlocked yes)
@@
 			)
 		)
-		(property "Value" "27k"
+		(property "Value" "2.7k"
 			(at 0 1.43 180)
 			(unlocked yes)
