File: circuit_ESP32C3_Xiao/ESP32C3_Xiao_wireless_DAP.kicad_sch (KiCad schematic)
At the start: 44 parts, among them J1 Cortex Debug 10pin connector, J2 ARM Standard JTAG, J3 Cortex Debug 10pin connector, J4 Conn_01x02, J6 Serial, Q1 YJL2304A, U1 XIAO-ESP32-C3-SMD, U2 AP1117-ADJ

Commit message: Update ESP32-C3 VTarget hardware design
Record the current ESP32-C3 XIAO schematic and PCB updates for the VTarget circuit.
Parts:
- C2: value 10nF -> 10uF /16V
- R4: value 39k -> 22k
- R5: value 10k -> 43k
Connections:
- net Vadj: now reaches C1.1, R1.2, R15.1, R3.1, U2.1 (ADJ)
Other:
- note added: "AO3400A"
- note added: "R4 - 40k || 39k R5 - 43k"
Changed lines of the file:
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@@
 		)
 	)
+	(text "R4 - 40k || 39k\nR5 - 43k"
+		(exclude_from_sim no)
+		(at 102.235 189.23 0)
+		(effects
+			(font
+				(size 1.27 1.27)
+			)
+		)
+	)
+	(text "AO3400A"
+		(exclude_from_sim no)
+		(at 118.11 184.912 0)
+		(effects
+			(font
+				(size 1.27 1.27)
+			)
+		)
+	)
 	(text ".param pulse_width = 0.1\n.param period = 20u\n; .dc pulse_width 0.1 0.9 0.1\n.OPTIONS METHOD=GEAR\n.OPTIONS RELTOL=0.01\n.OPTIONS VNTOL=10uV"
 		(exclude_from_sim no)
@@
 		)
 	)
+	(label "Vadj"
+		(at 119.38 142.24 0)
+		(effects
+			(font
+				(size 1.27 1.27)
+			)
+			(justify left bottom)
+		)
+	)
 	(label "TDI"
 		(at 196.85 45.72 180)
@@
 			)
 		)
-		(property "Value" "39k"
+		(property "Value" "22k"
 			(at 73.66 166.37 90)
 			(effects
@@
 		)
 		(instances
-			(project ""
+			(project "ESP32C3_Xiao_wireless_DAP"
 				(path "/ef31936a-2a92-40a9-b57a-332afb0572a5"
 					(reference "U2")
@@
 		)
 		(instances
-			(project ""
+			(project "ESP32C3_Xiao_wireless_DAP"
 				(path "/ef31936a-2a92-40a9-b57a-332afb0572a5"
 					(reference "#PWR03")
@@
 		)
 		(instances
-			(project ""
+			(project "ESP32C3_Xiao_wireless_DAP"
 				(path "/ef31936a-2a92-40a9-b57a-332afb0572a5"
 					(reference "H1")
@@
 		)
 		(instances
-			(project ""
+			(project "ESP32C3_Xiao_wireless_DAP"
 				(path "/ef31936a-2a92-40a9-b57a-332afb0572a5"
 					(reference "V1")
@@
 		)
 		(instances
-			(project ""
+			(project "ESP32C3_Xiao_wireless_DAP"
 				(path "/ef31936a-2a92-40a9-b57a-332afb0572a5"
 					(reference "J6")
@@
 		)
 		(instances
-			(project ""
+			(project "ESP32C3_Xiao_wireless_DAP"
 				(path "/ef31936a-2a92-40a9-b57a-332afb0572a5"
 					(reference "J1")
@@
 		)
 		(instances
-			(project ""
+			(project "ESP32C3_Xiao_wireless_DAP"
 				(path "/ef31936a-2a92-40a9-b57a-332afb0572a5"
 					(reference "V3")
@@
 		)
 		(instances
-			(project ""
+			(project "ESP32C3_Xiao_wireless_DAP"
 				(path "/ef31936a-2a92-40a9-b57a-332afb0572a5"
 					(reference "#PWR01")
@@
 		)
 		(instances
-			(project ""
+			(project "ESP32C3_Xiao_wireless_DAP"
 				(path "/ef31936a-2a92-40a9-b57a-332afb0572a5"
 					(reference "V2")
@@
 		)
 		(instances
-			(project ""
+			(project "ESP32C3_Xiao_wireless_DAP"
 				(path "/ef31936a-2a92-40a9-b57a-332afb0572a5"
 					(reference "U1")
@@
 		)
 		(instances
-			(project ""
+			(project "ESP32C3_Xiao_wireless_DAP"
 				(path "/ef31936a-2a92-40a9-b57a-332afb0572a5"
 					(reference "#PWR05")
@@
 		)
 		(instances
-			(project ""
+			(project "ESP32C3_Xiao_wireless_DAP"
 				(path "/ef31936a-2a92-40a9-b57a-332afb0572a5"
 					(reference "J2")
@@
 		)
 		(instances
-			(project ""
+			(project "ESP32C3_Xiao_wireless_DAP"
 				(path "/ef31936a-2a92-40a9-b57a-332afb0572a5"
 					(reference "Q1")
@@
 		)
 		(instances
-			(project ""
+			(project "ESP32C3_Xiao_wireless_DAP"
 				(path "/ef31936a-2a92-40a9-b57a-332afb0572a5"
 					(reference "D4")
@@
 			)
 		)
-		(property "Value" "10k"
+		(property "Value" "43k"
 			(at 97.79 176.5299 0)
 			(effects
@@
 		)
 		(instances
-			(project ""
+			(project "ESP32C3_Xiao_wireless_DAP"
 				(path "/ef31936a-2a92-40a9-b57a-332afb0572a5"
 					(reference "C1")
@@
 		)
 		(instances
-			(project ""
+			(project "ESP32C3_Xiao_wireless_DAP"
 				(path "/ef31936a-2a92-40a9-b57a-332afb0572a5"
 					(reference "D1")
@@
 		)
 		(instances
-			(project ""
+			(project "ESP32C3_Xiao_wireless_DAP"
 				(path "/ef31936a-2a92-40a9-b57a-332afb0572a5"
 					(reference "J4")
@@
 			)
 		)
-		(property "Value" "10nF"
+		(property "Value" "10uF /16V"
 			(at 107.95 176.5299 0)
 			(effects
@@
 		)
 		(instances
-			(project ""
+			(project "ESP32C3_Xiao_wireless_DAP"
 				(path "/ef31936a-2a92-40a9-b57a-332afb0572a5"
 					(reference "R1")

Commit message: Calibrate VTarget PWM control range
Map VTarget commands to the DMM-verified operating window, update the ESP32-C3 board values, refresh test curves, and document the calibration results.
Parts:
- C2: value 10uF /16V -> 10uF /25V
- R4: value 22k -> 100R
Changed lines of the file:
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@@
 			)
 		)
-		(property "Value" "22k"
+		(property "Value" "100R"
 			(at 73.66 166.37 90)
 			(effects
@@
 			)
 		)
-		(property "Value" "10uF /16V"
+		(property "Value" "10uF /25V"
 			(at 107.95 176.5299 0)
 			(effects

Commit message: Update KiCad schematic, PCB, and iBOM
Sync ESP32-C3 XIAO KiCad schematic, PCB, and interactive BOM with the R4/R5/C2 calibration hardware.
Parts:
- R1: value 12k -> 1.2k
- R3: value 27k -> 2.7k
- R4: value 100R -> 22k
Other:
- note removed: "R4 - 40k || 39k R5 - 43k"
Changed lines of the file:
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@@
 		)
 	)
-	(text "R4 - 40k || 39k\nR5 - 43k"
-		(exclude_from_sim no)
-		(at 102.235 189.23 0)
-		(effects
-			(font
-				(size 1.27 1.27)
-			)
-		)
-	)
 	(text "AO3400A"
 		(exclude_from_sim no)
@@
 			)
 		)
-		(property "Value" "100R"
+		(property "Value" "22k"
 			(at 73.66 166.37 90)
 			(effects
@@
 			)
 		)
-		(property "Value" "12k"
+		(property "Value" "1.2k"
 			(at 140.97 139.6999 0)
 			(effects
@@
 			)
 		)
-		(property "Value" "27k"
+		(property "Value" "2.7k"
 			(at 130.81 166.3699 0)
 			(effects
